Commit message: text

File: universal_robots_ws/src/my_universal_robots/my_ur_description/urdf/ur5/ur5_robot.urdf.xacro (robot description, xacro)
@@ -39,5 +39,5 @@
   <link name="baseplate_link">
     <visual>
-      <origin xyz="0 0 0.0" />
+      <origin xyz="0.35 0.55 -0.015" />
       <geometry>
         <box size="0.7 1.1 0.03" />
@@ -51,5 +51,5 @@
   </link>
   <joint name="baseplate_joint" type="fixed">
-    <origin xyz="0 0 0" />
+    <origin xyz="0.35 0.55 -0.015" />
     <parent link="world" />
     <child link="baseplate_link" />
@@ -57,5 +57,5 @@
   <link name="mountingplate_link">
     <visual>
-      <origin xyz="0 0 0.0" />
+      <origin xyz="0.15 0.15 0.006" rpy="0 0 3.14"/>
       <geometry>
         <box size="0.3 0.3 0.012" />
@@ -69,5 +69,5 @@
   </link>
   <joint name="mountingplate_joint" type="fixed">
-    <origin xyz="-0.2 0.0 0.021" />
+    <origin xyz="0.3 0.395 0.0" rpy="0 0 1.57" />
     <parent link="baseplate_link" />
     <child link="mountingplate_link" />
@@ -86,3 +86,193 @@
     <origin xyz="0.0 0.0 0.0" rpy="0.0 ${-pi/2} 0.0"/>
   </joint>
+  <!-- sorteerbakken -->
+  <link name="bak1_1_link">
+    <visual>
+      <origin xyz="0 0 0.001" rpy="1.57079 3.14 0.0"/>
+      <geometry>
+        <mesh filename="package://my_ur_description/urdf/ur5/sorteerbak_groot.STL"/>
+      </geometry>
+      <material name="blue"/>
+    </visual>
+    <collision>
+      <origin xyz="0 0 0.001" rpy="1.57079 3.14 0.0"/>
+      <geometry>
+        <mesh filename="package://my_ur_description/urdf/ur5/sorteerbak_groot.STL"/>
+      </geometry>
+      <material name="blue"/>
+    </collision>
+  </link>
+  <joint name="bak1_1_joint" type="fixed">
+    <origin xyz="0.102 1.15 0.082" />
+    <parent link="baseplate_link" />
+    <child link="bak1_1_link" />
+  </joint>
+  <link name="bak1_2_link">
+    <visual>
+      <origin xyz="0 0 0.001" rpy="1.57079 3.14 0.0"/>
+      <geometry>
+        <mesh filename="package://my_ur_description/urdf/ur5/sorteerbak_groot.STL"/>
+      </geometry>
+      <material name="blue"/>
+    </visual>
+    <collision>
+      <origin xyz="0 0 0.001" rpy="1.57079 3.14 0.0"/>
+      <geometry>
+        <mesh filename="package://my_ur_description/urdf/ur5/sorteerbak_groot.STL"/>
+      </geometry>
+      <material name="blue"/>
+    </collision>
+  </link>
+  <joint name="bak1_2_joint" type="fixed">
+    <origin xyz="0.105 0 0" />
+    <parent link="bak1_1_link" />
+    <child link="bak1_2_link" />
+  </joint>
+  <link name="bak1_3_link">
+    <visual>
+      <origin xyz="0 0 0.001" rpy="1.57079 3.14 0.0"/>
+      <geometry>
+        <mesh filename="package://my_ur_description/urdf/ur5/sorteerbak_groot.STL"/>
+      </geometry>
+      <material name="blue"/>
+    </visual>
+    <collision>
+      <origin xyz="0 0 0.001" rpy="1.57079 3.14 0.0"/>
+      <geometry>
+        <mesh filename="package://my_ur_description/urdf/ur5/sorteerbak_groot.STL"/>
+      </geometry>
+      <material name="blue"/>
+    </collision>
+  </link>
+  <joint name="bak1_3_joint" type="fixed">
+    <origin xyz="0.105 0 0" />
+    <parent link="bak1_2_link" />
+    <child link="bak1_3_link" />
+  </joint>
+  <link name="bak1_4_link">
+    <visual>
+      <origin xyz="0 0 0.001" rpy="1.57079 3.14 0.0"/>
+      <geometry>
+        <mesh filename="package://my_ur_description/urdf/ur5/sorteerbak_groot.STL"/>
+      </geometry>
+      <material name="blue"/>
+    </visual>
+    <collision>
+      <origin xyz="0 0 0.001" rpy="1.57079 3.14 0.0"/>
+      <geometry>
+        <mesh filename="package://my_ur_description/urdf/ur5/sorteerbak_groot.STL"/>
+      </geometry>
+      <material name="blue"/>
+    </collision>
+  </link>
+  <joint name="bak1_4_joint" type="fixed">
+    <origin xyz="0.105 0 0" />
+    <parent link="bak1_3_link" />
+    <child link="bak1_4_link" />
+  </joint>
+  <link name="bak2_1_link">
+    <visual>
+      <origin xyz="0 0 0.001" rpy="1.57079 3.14 0.0"/>
+      <geometry>
+        <mesh filename="package://my_ur_description/urdf/ur5/sorteerbak_klein.STL"/>
+      </geometry>
+      <material name="blue"/>
+    </visual>
+    <collision>
+      <origin xyz="0 0 0.001" rpy="1.57079 3.14 0.0"/>
+      <geometry>
+        <mesh filename="package://my_ur_description/urdf/ur5/sorteerbak_klein.STL"/>
+      </geometry>
+      <material name="blue"/>
+    </collision>
+  </link>
+  <joint name="bak2_1_joint" type="fixed">
+    <origin xyz="-0.102 0 0.002" rpy="0.0 3.14 0.0"  />
+    <parent link="bak1_1_link" />
+    <child link="bak2_1_link" />
+  </joint>
+  <link name="bak2_2_link">
+    <visual>
+      <origin xyz="0 0 0.001" rpy="1.57079 3.14 0.0"/>
+      <geometry>
+        <mesh filename="package://my_ur_description/urdf/ur5/sorteerbak_klein.STL"/>
+      </geometry>
+      <material name="blue"/>
+    </visual>
+    <collision>
+      <origin xyz="0 0 0.001" rpy="1.57079 3.14 0.0"/>
+      <geometry>
+        <mesh filename="package://my_ur_description/urdf/ur5/sorteerbak_klein.STL"/>
+      </geometry>
+      <material name="blue"/>
+    </collision>
+  </link>
+  <joint name="bak2_2_joint" type="fixed">
+    <origin xyz="-0.105 0 0" rpy="0.0 0 0.0"  />
+    <parent link="bak2_1_link" />
+    <child link="bak2_2_link" />
+  </joint>
+  <link name="bak2_3_link">
+    <visual>
+      <origin xyz="0 0 0.001" rpy="1.57079 3.14 0.0"/>
+      <geometry>
+        <mesh filename="package://my_ur_description/urdf/ur5/sorteerbak_klein.STL"/>
+      </geometry>
+      <material name="blue"/>
+    </visual>
+    <collision>
+      <origin xyz="0 0 0.001" rpy="1.57079 3.14 0.0"/>
+      <geometry>
+        <mesh filename="package://my_ur_description/urdf/ur5/sorteerbak_klein.STL"/>
+      </geometry>
+      <material name="blue"/>
+    </collision>
+  </link>
+  <joint name="bak2_3_joint" type="fixed">
+    <origin xyz="-0.105 0 0" rpy="0.0 0 0.0"  />
+    <parent link="bak2_2_link" />
+    <child link="bak2_3_link" />
+  </joint>
+  <link name="bak2_4_link">
+    <visual>
+      <origin xyz="0 0 0.001" rpy="1.57079 3.14 0.0"/>
+      <geometry>
+        <mesh filename="package://my_ur_description/urdf/ur5/sorteerbak_klein.STL"/>
+      </geometry>
+      <material name="blue"/>
+    </visual>
+    <collision>
+      <origin xyz="0 0 0.001" rpy="1.57079 3.14 0.0"/>
+      <geometry>
+        <mesh filename="package://my_ur_description/urdf/ur5/sorteerbak_klein.STL"/>
+      </geometry>
+      <material name="blue"/>
+    </collision>
+  </link>
+  <joint name="bak2_4_joint" type="fixed">
+    <origin xyz="-0.105 0 0" rpy="0.0 0 0.0"  />
+    <parent link="bak2_3_link" />
+    <child link="bak2_4_link" />
+  </joint>
+  <link name="transportsystem_link">
+    <visual>
+      <origin xyz="0 0 0" rpy=" 0 0 0"/>
+      <geometry>
+        <mesh filename="package://my_ur_description/urdf/ur5/transportsystem.STL"/>
+      </geometry>
+      <material name="blue"/>
+    </visual>
+    <collision>
+      <origin xyz="0 0 0" rpy="0 0 0"/>
+      <geometry>
+        <mesh filename="package://my_ur_description/urdf/ur5/transportsystem.STL"/>
+      </geometry>
+      <material name="blue"/>
+    </collision>
+  </link>
+  <joint name="transportsystem_joint" type="fixed">
+    <origin xyz="0.02 0.32 0" rpy=" 1.57 0 0"/>
+    <parent link="baseplate_link" />
+    <child link="transportsystem_link" />
+  </joint>
 </robot>

Commit message: transportsysteem:
-transportsysteem toegevoegd aan RVIZ

File: universal_robots_ws/src/my_universal_robots/my_ur_description/urdf/ur5/ur5_robot.urdf.xacro (robot description, xacro)
@@ -276,3 +276,24 @@
     <child link="grippervision_link" />
   </joint>
+ <link name="transportsystem_link">
+    <visual>
+      <origin xyz="0 0 0" rpy=" 0 0 0"/>
+      <geometry>
+        <mesh filename="package://my_ur_description/urdf/ur5/transportsystem.STL"/>
+      </geometry>
+      <material name="blue"/>
+    </visual>
+    <collision>
+      <origin xyz="0 0 0" rpy="0 0 0"/>
+      <geometry>
+        <mesh filename="package://my_ur_description/urdf/ur5/transportsystem.STL"/>
+      </geometry>
+      <material name="blue"/>
+    </collision>
+  </link>
+  <joint name="transportsystem_joint" type="fixed">
+    <origin xyz="0.02 0.32 0" rpy=" 1.57 0 0"/>
+    <parent link="baseplate_link" />
+    <child link="transportsystem_link" />
+  </joint>
 </robot>

Commit message: hoofdprogramma update

File: universal_robots_ws/src/my_universal_robots/my_ur_description/urdf/ur5/ur5_robot.urdf.xacro (robot description, xacro)
@@ -104,5 +104,5 @@
   </link>
   <joint name="bak1_1_joint" type="fixed">
-    <origin xyz="0.102 1.15 0.082" />
+    <origin xyz="0.102 1.1 0.082" />
     <parent link="baseplate_link" />
     <child link="bak1_1_link" />
@@ -293,5 +293,5 @@
   </link>
   <joint name="transportsystem_joint" type="fixed">
-    <origin xyz="0.02 0.32 0" rpy=" 1.57 0 0"/>
+    <origin xyz="0.02 0.38 0" rpy=" 1.57 0 0"/>
     <parent link="baseplate_link" />
     <child link="transportsystem_link" />
